File: Circuit_Schematic/senior_design.sch (EAGLE design)
At the start: 17 parts, among them IC1 INA118P

Commit message: updates
Parts:
- added C4, C5, C6, C7, C8: (no value), capacitor-wima:C2,5-3
- added IC2: TLC272P, linear:TLC272P
Changed lines of the file:
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@@
 <part name="D4" library="diode" library_urn="urn:adsk.eagle:library:210" deviceset="1N4148" device="DO35-7" package3d_urn="urn:adsk.eagle:package:43339/1" value=""/>
 <part name="IC1" library="burr-brown" library_urn="urn:adsk.eagle:library:111" deviceset="INA118" device="P" package3d_urn="urn:adsk.eagle:package:4906/1"/>
+<part name="C4" library="capacitor-wima" library_urn="urn:adsk.eagle:library:116" deviceset="C" device="2,5-3" package3d_urn="urn:adsk.eagle:package:5436/1"/>
+<part name="C5" library="capacitor-wima" library_urn="urn:adsk.eagle:library:116" deviceset="C" device="2,5-3" package3d_urn="urn:adsk.eagle:package:5436/1"/>
+<part name="C6" library="capacitor-wima" library_urn="urn:adsk.eagle:library:116" deviceset="C" device="2,5-3" package3d_urn="urn:adsk.eagle:package:5436/1"/>
+<part name="C7" library="capacitor-wima" library_urn="urn:adsk.eagle:library:116" deviceset="C" device="2,5-3" package3d_urn="urn:adsk.eagle:package:5436/1"/>
+<part name="C8" library="capacitor-wima" library_urn="urn:adsk.eagle:library:116" deviceset="C" device="2,5-3" package3d_urn="urn:adsk.eagle:package:5436/1"/>
+<part name="IC2" library="linear" library_urn="urn:adsk.eagle:library:262" deviceset="TLC272" device="P" package3d_urn="urn:adsk.eagle:package:16409/2"/>
 </parts>
 <sheets>
@@
 <instance part="D4" gate="G$1" x="48.26" y="7.62" rot="R90"/>
 <instance part="IC1" gate="G$1" x="88.9" y="45.72"/>
+<instance part="C4" gate="G$1" x="109.22" y="50.8"/>
+<instance part="C5" gate="G$1" x="127" y="45.72"/>
+<instance part="C6" gate="G$1" x="162.56" y="66.04"/>
+<instance part="C7" gate="G$1" x="160.02" y="27.94"/>
+<instance part="C8" gate="G$1" x="147.32" y="45.72"/>
+<instance part="IC2" gate="A" x="129.54" y="58.42"/>
+<instance part="IC2" gate="B" x="162.56" y="45.72"/>
 </instances>
 <busses>
