File: PCB/senior_design.sch (EAGLE design)
At the start: 21 parts, among them IC1 LF356N, IC2 LF356N, IC3 LM741P, IC4 LM741P

Commit message: updates
Connections:
- net PE renamed VO
- net N$3: no longer R7.1
- net N$8: now also R7.1
Changed lines of the file:
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@@
 <wire x1="45.72" y1="68.58" x2="30.48" y2="68.58" width="0.1524" layer="91"/>
 <junction x="30.48" y="68.58"/>
-<pinref part="R7" gate="G$1" pin="1"/>
-<wire x1="45.72" y1="68.58" x2="73.66" y2="68.58" width="0.1524" layer="91"/>
-<junction x="45.72" y="68.58"/>
 </segment>
 </net>
@@
 <pinref part="IC3" gate="A" pin="-IN"/>
 <wire x1="55.88" y1="38.1" x2="63.5" y2="38.1" width="0.1524" layer="91"/>
+<pinref part="R7" gate="G$1" pin="1"/>
+<wire x1="73.66" y1="68.58" x2="55.88" y2="68.58" width="0.1524" layer="91"/>
+<wire x1="55.88" y1="68.58" x2="55.88" y2="38.1" width="0.1524" layer="91"/>
+<junction x="55.88" y="38.1"/>
 </segment>
 </net>
@@
 </segment>
 </net>
-<net name="N$15" class="0">
-<segment>
-<pinref part="R11" gate="G$1" pin="2"/>
-<wire x1="149.86" y1="38.1" x2="154.94" y2="38.1" width="0.1524" layer="91"/>
-<pinref part="C2" gate="G$1" pin="1"/>
-<wire x1="154.94" y1="38.1" x2="154.94" y2="33.02" width="0.1524" layer="91"/>
-</segment>
-</net>
 <net name="N$17" class="0">
 <segment>
@@
 </segment>
 </net>
-<net name="PE" class="0">
+<net name="VO" class="0">
 <segment>
 <pinref part="R6" gate="G$1" pin="1"/>
@@
 </segment>
 </net>
+<net name="N$9" class="0">
+<segment>
+<pinref part="R11" gate="G$1" pin="2"/>
+<wire x1="149.86" y1="38.1" x2="154.94" y2="38.1" width="0.1524" layer="91"/>
+<pinref part="C2" gate="G$1" pin="1"/>
+<wire x1="154.94" y1="38.1" x2="154.94" y2="33.02" width="0.1524" layer="91"/>
+</segment>
+</net>
