File: PCB/senior_design.brd (EAGLE design)
At the start: 100 x 80 mm, 20 parts, among them IC1 LF356N, IC2 LF356N, IC3 LM741P, IC4 LM741P

Commit message: updates
Connections:
- net PE renamed VO
- net N$3: no longer R7.1
- net N$8: now also R7.1
Routing:
- net V+: track 68.0 -> 95.8 mm
- net VO: track 21.8 -> 6.13 mm, vias 0 -> 1
- net N$8: track 8.06 -> 19.7 mm
- net N$12: track 10.5 -> 16.3 mm
- net N$3: track 21.4 -> 16.2 mm
- net N$11: track 19.8 -> 24.7 mm
- net V-: track 62.3 -> 66.8 mm
- net N$10: track 23.3 -> 25.8 mm
- net N$9: track 22.1 -> 23.9 mm
- net N$7: track 20.1 -> 21.7 mm
- net N$13: track 16.8 -> 18.3 mm
Other:
- board text added: "C1"
- board text added: "C2"
- board text added: "C3"
- board text added: "C4"
- board text added: "IC1"
- board text added: "IC2"
- board text added: "IC3"
- board text added: "IC4"
- board text added: "R1"
- board text added: "R10"
- board text added: "R11"
- board text added: "R12"
- board text added: "R2"
- board text added: "R3"
- board text added: "R4"
- board text added: "R5"
- board text added: "R6"
- board text added: "R7"
- board text added: "R8"
- board text added: "R9"
